File: kicad/GPS_CLock/GPS_CLock.kicad_pcb (KiCad board)
At the start: 4 copper layers, 449.5 x 33 mm, 181 parts, among them J101 SWD, J102 UART, J201 USB_C_2.0, J401 U.FL, J501 1-1734839-6, SW101 BOOT_JMP, SW102 SW_Push, SW103 SW_Push, U101 W25Q16JVUXIQ, U102 VEML7700-TR, U103 RP2040, U104 MS8607, U201 LP5912-3.3DRV, U202 STUSB4500QTR, U204 TPS62827DMQ, U205 TPS62827DMQ, U301 DG0, U302 DG1, U303 LED_CC7, U304 LED_CC6, U305 DG2, U306 DG3, U307 74AUP2G17, U308 74AUP2G17, U309 DG4, U310 DG5, U311 LED_CC8, U312 LED_CC5, U313 DG6, U314 DG7, U315 DG8, U316 DG9, U317 LED_CC9, U318 LED_CC4, U319 DG10, U320 74AUP2G17, U321 DG11, U322 74AUP2G17, U323 DG12, U324 LED_CC10, U325 LED_CC3, U326 DG13, U327 DG14, U328 DG15, U329 LED_CC11, U330 LED_CC2, U331 DG16, U332 DG17, U333 74AUP2G17, U334 74AUP2G17, U335 DG18, U336 DG19, U337 LED_CC12, U338 LED_CC1, U339 DG20, U340 DG21, U341 DG22, U342 LED_CC13, U343 LED_CC0, U344 DG23, U345 DG24, U401 MAX-M10S

Commit message: updated pcb
Parts:
- added C203: 1u, Capacitor_SMD:C_0402_1005Metric, B.Cu at (455.5, 168.7)
- added C205: 1u, Capacitor_SMD:C_0402_1005Metric, B.Cu at (451.9, 168.7)
- added C206: 1u, Capacitor_SMD:C_0402_1005Metric, B.Cu at (453.7, 168.7)
- added C212: 47n, Capacitor_SMD:C_0402_1005Metric, B.Cu at (444.9, 164.3)
- added C501: 10u, Capacitor_SMD:C_0402_1005Metric, F.Cu at (453.7, 141.0)
- added C504: 10u, Capacitor_SMD:C_0402_1005Metric, F.Cu at (453.7, 143.0)
- added D201: BAT54, Diode_SMD:D_SOD-323, B.Cu at (455.3, 162.8)
- added Q201: PMPB17EP, clock:NXP_DFN6_2.0x2.0mm 2xEp, B.Cu at (455.3, 165.7)
- added Q202: PMPB17EP, clock:NXP_DFN6_2.0x2.0mm 2xEp, B.Cu at (453.0, 165.7)
- added R205: 100, Resistor_SMD:R_0402_1005Metric, B.Cu at (453.4, 162.9)
- added R501: 680k, Resistor_SMD:R_0402_1005Metric, F.Cu at (450.9, 141.0)
- added R502: 5.1k, Resistor_SMD:R_0402_1005Metric, F.Cu at (450.9, 143.0)
- added U203: BQ25892, Package_DFN_QFN:Texas_S-PWQFN-N24_EP2.7x2.7mm, B.Cu at (445.8, 167.9)
- C202, C207, C210, C211, C213, C215, C216, HSE101, J401, R103, R104, R201, R202, R204, R206, R211, R212, R215, R216, SW102, U101, U103, U202, U204, U205, U337, U342, U343, U401: moved to B.Cu
- C208, C209, C217, C218, C219, C221: footprint Capacitor_SMD:C_0402_1005Metric -> Capacitor_SMD:C_0603_1608Metric; moved to B.Cu
- L201, L202: footprint Inductor_SMD:L_0805_2012Metric -> clock:L_DFE201610; moved to B.Cu
- L203: footprint clock:Bourns_SRP2512 -> Inductor_SMD:L_Vishay_IHLP-2020; moved to B.Cu
- moved H105 307.6 mm to (461.0, 155.0)
- moved H106 304.5 mm to (461.0, 181.0)
- moved U302 280.6 mm to (46.0, 168.0)
- moved U301 263.8 mm to (29.0, 168.0)
- moved U344 249.9 mm to (429.0, 168.0)
- moved R104 244.8 mm to (432.9, 169.4), turned to 180 degrees
- moved U103 242.9 mm to (427.0, 171.0), turned to 90 degrees
- moved D306 238.9 mm to (417.0, 173.0), turned to 90 degrees
- moved U305 236.2 mm to (63.0, 168.0)
- moved R103 231.7 mm to (432.9, 170.3), turned to 180 degrees
- moved D305 231.2 mm to (417.0, 162.0), turned to -90 degrees
- moved HSE101 228.9 mm to (420.5, 170.5), turned to -90 degrees
- moved U101 225.0 mm to (433.5, 174.5), turned to 180 degrees
- moved U319 219.4 mm to (196.0, 168.0)
- moved SW102 208.4 mm to (396.5, 151.5)
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Connections:
- net Net-(C207-Pad1) renamed /Power/VBUS_SNK
- net Net-(D201-Pad2) renamed /Power/VBUS
- D301 pad 2: /Segments/SEG_2.5V_BOT -> SEG_2.5V_BOT
- D302 pad 2: /Segments/SEG_2.5V_BOT -> SEG_2.5V_BOT
- D303 pad 2: /Segments/SEG_2.5V_BOT -> SEG_2.5V_BOT
- D304 pad 2: /Segments/SEG_2.5V_BOT -> SEG_2.5V_BOT
- D305 pad 2: /Segments/SEG_2.5V_BOT -> SEG_2.5V_BOT
- D306 pad 2: /Segments/SEG_2.5V_BOT -> SEG_2.5V_BOT
- U103 pad 6: /LED_MOSI -> /SEG_MOSI
- U103 pad 7: /LED_LAT -> /SEG_LAT
- U103 pad 8: /LED_SCK -> /SEG_CLK
- U103 pad 9: /LED_OE -> /SEG_OE
- U202 pad 7: unconnected-(U202-Pad7) -> /POW_SCL
- U202 pad 8: unconnected-(U202-Pad8) -> /POW_SDA
- U301 pad 1: /Segments/SEG_2.5V_BOT -> SEG_2.5V_BOT
- U301 pad 6: /Segments/SEG_2.5V_TOP -> SEG_2.5V_TOP
- U302 pad 1: /Segments/SEG_2.5V_BOT -> SEG_2.5V_BOT
- U302 pad 6: /Segments/SEG_2.5V_TOP -> SEG_2.5V_TOP
- U303 pad 24: /Segments/SEG_OE_CONN -> /SEG_OE
- U304 pad 24: /Segments/SEG_OE_CONN -> /SEG_OE
- U305 pad 1: /Segments/SEG_2.5V_BOT -> SEG_2.5V_BOT
- U305 pad 6: /Segments/SEG_2.5V_TOP -> SEG_2.5V_TOP
- U306 pad 1: /Segments/SEG_2.5V_BOT -> SEG_2.5V_BOT
- U306 pad 6: /Segments/SEG_2.5V_TOP -> SEG_2.5V_TOP
- U309 pad 1: /Segments/SEG_2.5V_BOT -> SEG_2.5V_BOT
- U309 pad 6: /Segments/SEG_2.5V_TOP -> SEG_2.5V_TOP
- U310 pad 1: /Segments/SEG_2.5V_BOT -> SEG_2.5V_BOT
- U310 pad 6: /Segments/SEG_2.5V_TOP -> SEG_2.5V_TOP
- U311 pad 24: /Segments/SEG_OE_CONN -> /SEG_OE
- U312 pad 24: /Segments/SEG_OE_CONN -> /SEG_OE
- U313 pad 1: /Segments/SEG_2.5V_BOT -> SEG_2.5V_BOT
- U313 pad 6: /Segments/SEG_2.5V_TOP -> SEG_2.5V_TOP
- U314 pad 1: /Segments/SEG_2.5V_BOT -> SEG_2.5V_BOT
- U314 pad 6: /Segments/SEG_2.5V_TOP -> SEG_2.5V_TOP
- U315 pad 1: /Segments/SEG_2.5V_BOT -> SEG_2.5V_BOT
- U315 pad 6: /Segments/SEG_2.5V_TOP -> SEG_2.5V_TOP
- U316 pad 1: /Segments/SEG_2.5V_BOT -> SEG_2.5V_BOT
- U316 pad 6: /Segments/SEG_2.5V_TOP -> SEG_2.5V_TOP
- U317 pad 24: /Segments/SEG_OE_CONN -> /SEG_OE
- U318 pad 24: /Segments/SEG_OE_CONN -> /SEG_OE
- U319 pad 14: /Segments/SEG_2.5V_TOP -> SEG_2.5V_TOP
- U321 pad 1: /Segments/SEG_2.5V_BOT -> SEG_2.5V_BOT
- U321 pad 6: /Segments/SEG_2.5V_TOP -> SEG_2.5V_TOP
- U323 pad 1: /Segments/SEG_2.5V_BOT -> SEG_2.5V_BOT
- U323 pad 6: /Segments/SEG_2.5V_TOP -> SEG_2.5V_TOP
- U324 pad 24: /Segments/SEG_OE_CONN -> /SEG_OE
- U325 pad 24: /Segments/SEG_OE_CONN -> /SEG_OE
- U326 pad 1: /Segments/SEG_2.5V_BOT -> SEG_2.5V_BOT
- U326 pad 6: /Segments/SEG_2.5V_TOP -> SEG_2.5V_TOP
- U327 pad 1: /Segments/SEG_2.5V_BOT -> SEG_2.5V_BOT
- U327 pad 6: /Segments/SEG_2.5V_TOP -> SEG_2.5V_TOP
- U328 pad 1: /Segments/SEG_2.5V_BOT -> SEG_2.5V_BOT
- U328 pad 6: /Segments/SEG_2.5V_TOP -> SEG_2.5V_TOP
- U329 pad 24: /Segments/SEG_OE_CONN -> /SEG_OE
- U330 pad 24: /Segments/SEG_OE_CONN -> /SEG_OE
- U331 pad 1: /Segments/SEG_2.5V_BOT -> SEG_2.5V_BOT
- U331 pad 6: /Segments/SEG_2.5V_TOP -> SEG_2.5V_TOP
- U332 pad 1: /Segments/SEG_2.5V_BOT -> SEG_2.5V_BOT
- U332 pad 6: /Segments/SEG_2.5V_TOP -> SEG_2.5V_TOP
- U334 pad 1: /Segments/SEG_CLK_CONN -> /SEG_CLK
- U334 pad 3: /Segments/SEG_LAT_CONN -> /SEG_LAT
- U335 pad 1: /Segments/SEG_2.5V_BOT -> SEG_2.5V_BOT
- U335 pad 6: /Segments/SEG_2.5V_TOP -> SEG_2.5V_TOP
- U336 pad 1: /Segments/SEG_2.5V_BOT -> SEG_2.5V_BOT
- U336 pad 6: /Segments/SEG_2.5V_TOP -> SEG_2.5V_TOP
- U337 pad 24: /Segments/SEG_OE_CONN -> /SEG_OE
- U338 pad 24: /Segments/SEG_OE_CONN -> /SEG_OE
- U338 pad 6: /Segments/SEG_CLK_CONN -> /SEG_CLK
- U338 pad 7: /Segments/SEG_LAT_CONN -> /SEG_LAT
- U338 pad 8: /Segments/DG21_E -> /Segments/DG21_D
- U339 pad 14: /Segments/SEG_2.5V_TOP -> SEG_2.5V_TOP
- U340 pad 1: /Segments/SEG_2.5V_BOT -> SEG_2.5V_BOT
- U340 pad 6: /Segments/SEG_2.5V_TOP -> SEG_2.5V_TOP
- U341 pad 1: /Segments/SEG_2.5V_BOT -> SEG_2.5V_BOT
- U341 pad 6: /Segments/SEG_2.5V_TOP -> SEG_2.5V_TOP
- U342 pad 11: /Segments/DG22_G -> /Segments/DG21_A
- U342 pad 12: /Segments/DG22_F -> /Segments/DG22_G
- U342 pad 13: /Segments/DG22_A -> /Segments/DG22_F
- U342 pad 15: /Segments/DG23_G -> /Segments/DG22_A
- U342 pad 16: /Segments/DG23_F -> /Segments/DG23_G
- U342 pad 17: /Segments/DG23_A -> /Segments/DG23_F
- U342 pad 19: /Segments/DG24_G -> /Segments/DG23_A
- U342 pad 20: /Segments/DG24_F -> /Segments/DG24_G
- U342 pad 21: /Segments/DG24_A -> /Segments/DG24_F
- U342 pad 23: /Segments/COL2_T -> /Segments/DG24_A
- U342 pad 24: /Segments/SEG_OE_CONN -> /SEG_OE
- U342 pad 8: /Segments/DG21_F -> /Segments/COL2_T
- U342 pad 9: /Segments/DG21_A -> /Segments/DG21_F
- U343 pad 10: /Segments/DG24_D -> /Segments/DG24_E
- U343 pad 11: /Segments/DG24_E -> /Segments/DG24_D
- U343 pad 14: /Segments/DG23_D -> /Segments/DG23_E
- U343 pad 15: /Segments/DG23_E -> /Segments/DG23_D
- U343 pad 16: /Segments/COL2_B -> /Segments/DG22_DP
- U343 pad 17: /Segments/DG22_DP -> /Segments/DG22_C
- U343 pad 18: /Segments/DG22_C -> /Segments/DG22_E
- U343 pad 20: /Segments/DG22_E -> /Segments/DG21_DP
- U343 pad 21: /Segments/DG21_DP -> /Segments/DG21_C
- U343 pad 22: /Segments/DG21_C -> /Segments/DG21_E
- U343 pad 23: /Segments/DG21_D -> /Segments/COL2_B
- U343 pad 24: /Segments/SEG_OE_CONN -> /SEG_OE
- U343 pad 5: /Segments/SEG_SOUT_CONN -> /SEG_MOSI
- U343 pad 6: /Segments/SEG_CLK_CONN -> /SEG_CLK
- U343 pad 7: /Segments/SEG_LAT_CONN -> /SEG_LAT
- U344 pad 1: /Segments/SEG_2.5V_BOT -> SEG_2.5V_BOT
- U344 pad 6: /Segments/SEG_2.5V_TOP -> SEG_2.5V_TOP
- U345 pad 1: /Segments/SEG_2.5V_BOT -> SEG_2.5V_BOT
- U345 pad 6: /Segments/SEG_2.5V_TOP -> SEG_2.5V_TOP
Routing:
- net /Segments/DG24_DP: track 0.00 -> 33.4 mm, vias 0 -> 1
- net /Segments/DG24_A: track 0.00 -> 30.7 mm, vias 0 -> 1
- net /Segments/DG21_F: track 0.00 -> 30.7 mm, vias 0 -> 1
- net /Segments/DG24_C: track 0.00 -> 30.4 mm, vias 0 -> 1
- net /Segments/DG24_B: track 0.00 -> 28.0 mm, vias 0 -> 1
- net /Segments/DG21_E: track 0.00 -> 27.8 mm, vias 0 -> 1
- net /Segments/DG21_B: track 0.00 -> 27.7 mm, vias 0 -> 1
- net /Segments/DG24_E: track 0.00 -> 27.5 mm, vias 0 -> 1
- net /Segments/DG18_F: track 0.00 -> 26.7 mm, vias 0 -> 1
- net /Segments/DG24_F: track 0.00 -> 25.2 mm, vias 0 -> 1
- net /Segments/DG21_C: track 0.00 -> 25.0 mm, vias 0 -> 1
- net /Segments/DG21_A: track 0.00 -> 24.9 mm, vias 0 -> 1
- net /Segments/DG24_D: track 0.00 -> 24.8 mm, vias 0 -> 1
- net /Segments/DG18_B: track 0.00 -> 23.1 mm, vias 0 -> 1
- net /Segments/DG24_G: track 0.00 -> 22.5 mm, vias 0 -> 1
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- added copper zone on In1.Cu, net +3V3
- added copper zone on In1.Cu, net +BATT
- added copper zone on B.Cu, net /Power/VBUS
- added copper zone on B.Cu, net /Power/VBUS_SNK
- added copper zone on B.Cu, net /Power/VSYS
- added copper zone on B.Cu, net Earth
- added copper zone on B.Cu, net Net-(C203-Pad2)
- added copper zone on B.Cu, net Net-(C212-Pad1)
- added copper zone on B.Cu, net Net-(L201-Pad1)
- added copper zone on B.Cu, net Net-(L202-Pad1)
- added copper zone on In1.Cu, net SEG_2.5V_BOT
- added copper zone on B.Cu, net SEG_2.5V_TOP
- added copper zone on F.Cu, net SEG_2.5V_TOP
- added copper zone on In1.Cu, net SEG_2.5V_TOP
Other:
- board size 449.5 x 33 mm -> 451 x 33 mm

Commit message: update pcb
Parts:
- added AE401: Active, Capacitor_SMD:C_0603_1608Metric, F.Cu at (463.4, 146.3)
- C201, C220: footprint Capacitor_SMD:C_0402_1005Metric -> Capacitor_SMD:C_0603_1608Metric; moved to B.Cu
- C204, C214, R203, R213, R214, U201: moved to B.Cu
- moved R214 71.8 mm to (452.3, 179.2), turned to -90 degrees
- moved R213 71.4 mm to (454.2, 179.2), turned to 90 degrees
- moved C220 67.9 mm to (450.4, 179.5)
- moved C214 65.9 mm to (453.2, 179.2), turned to 90 degrees
- moved C204 55.0 mm to (458.8, 157.8), turned to 180 degrees
- moved C201 54.1 mm to (456.2, 159.6), turned to -90 degrees
- moved R203 46.4 mm to (460.1, 159.6), turned to -90 degrees
- moved U201 17.6 mm to (458.3, 159.6), turned to 180 degrees
- moved C216 10.5 mm to (440.9, 160.0), turned to 90 degrees
- moved C217 9.60 mm to (442.1, 159.9), turned to 90 degrees
- moved R215 8.68 mm to (439.9, 163.8), turned to 0 degrees
- moved R216 8.40 mm to (439.9, 164.8), turned to 180 degrees
- moved R206 8.34 mm to (439.9, 165.7), turned to 180 degrees
- moved L203 7.43 mm to (447.9, 160.5), turned to 90 degrees
- moved C218 7.25 mm to (444.3, 160.7), turned to 0 degrees
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Routing:
- net USB_D-: track 2.67 -> 28.4 mm
- net USB_D+: track 0.50 -> 26.2 mm
- net SEG_2.5V_TOP: track 2.14 -> 19.4 mm, vias 13 -> 23
- net /BTN_DWN: track 0.00 -> 5.39 mm, vias 0 -> 2
- net +3V3: track 1.75 -> 6.64 mm, vias 1 -> 3
- net Earth: track 3.90 -> 7.14 mm, vias 14 -> 20
- net /Power/VBUS_SNK: track 0.00 -> 3.09 mm
- net Net-(C213-Pad2): track 0.00 -> 2.85 mm
- net Net-(C214-Pad2): track 0.00 -> 2.81 mm
- net SEG_2.5V_BOT: track 0.00 -> 2.04 mm, vias 0 -> 2
- net /Power/VSYS: track 0.00 -> 1.97 mm, vias 0 -> 15
- net Net-(C203-Pad2): track 6.17 -> 7.44 mm
- net /Segments/DG24_D: track 24.8 -> 25.7 mm
- net /Segments/DG24_A: track 30.7 -> 30.2 mm
- net /Power/VBUS: track 3.39 -> 3.35 mm, vias 0 -> 12
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- added copper zone on B.Cu, net +BATT
- added copper zone on In1.Cu, net /Power/VBUS
- added copper zone on F.Cu, net /Power/VSYS
- removed copper zone on F.Cu, net SEG_2.5V_TOP

Commit message: update pcb
Parts:
- moved L203 1.00 mm to (448.9, 160.5)
- moved C209 0.30 mm to (449.3, 177.3)
- moved C214 0.30 mm to (452.9, 179.2)
- moved C220 0.30 mm to (450.1, 179.5)
- moved L202 0.30 mm to (447.4, 178.3)
- moved R213 0.30 mm to (453.9, 179.2)
- moved R214 0.30 mm to (452.0, 179.2)
- moved U205 0.30 mm to (451.1, 177.3)
Routing:
- net SEG_2.5V_TOP: track 19.4 -> 7.87 mm, vias 23 -> 31
- net Earth: vias 20 -> 25
- net /Power/VBUS: vias 12 -> 13

Commit message: update pcb
Parts:
- C101, C102, C103, C105, C106, C107, C109, C110, C111, C112, C113, J501, R102, R208, R209, R210: moved to B.Cu
- moved R102 248.0 mm to (438.5, 172.5), turned to -90 degrees
- moved C103 244.0 mm to (451.8, 176.0), turned to 180 degrees
- moved C110 243.4 mm to (449.8, 167.7)
- moved C112 243.0 mm to (447.8, 166.6)
- moved C111 239.8 mm to (449.8, 171.2)
- moved C102 238.4 mm to (437.5, 172.5), turned to 90 degrees
- moved C107 237.1 mm to (449.8, 169.6)
- moved C101 235.9 mm to (437.5, 174.5), turned to -90 degrees
- moved C109 235.3 mm to (449.8, 168.7)
- moved C106 234.0 mm to (449.8, 172.1)
- moved C105 223.7 mm to (439.0, 170.0), turned to 180 degrees
- moved C113 222.8 mm to (439.0, 171.0), turned to 180 degrees
- moved J501 186.9 mm to (417.0, 165.3)
- moved R208 71.8 mm to (445.6, 177.2), turned to -90 degrees
- moved R210 65.8 mm to (460.6, 171.7), turned to -90 degrees
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Routing:
- net Earth: track 7.14 -> 46.2 mm, vias 25 -> 63
- net USB_D-: track 28.4 -> 2.67 mm
- net USB_D+: track 26.2 -> 0.50 mm
- net +3V3: track 6.64 -> 26.3 mm, vias 3 -> 20
- net +1V1: track 0.00 -> 11.5 mm, vias 0 -> 4
- net /XIN: track 0.00 -> 9.16 mm
- net Net-(R209-Pad2): track 0.00 -> 7.80 mm, vias 0 -> 2
- net /QSPI_SD3: track 0.00 -> 7.63 mm
- net Net-(C215-Pad1): track 1.17 -> 8.29 mm, vias 0 -> 2
- net /QSPI_SCLK: track 0.00 -> 6.49 mm
- net SEG_2.5V_TOP: track 7.87 -> 12.9 mm, vias 31 -> 23
- net /Power/TS: track 2.04 -> 6.87 mm, vias 0 -> 2
- net /QSPI_SD0: track 0.00 -> 4.61 mm
- net SEG_2.5V_BOT: track 2.04 -> 5.48 mm, vias 2 -> 0
- net Net-(R103-Pad2): track 0.00 -> 3.32 mm
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- added copper zone on B.Cu, net +1V1
- added copper zone on B.Cu, net +3V3
Other:
- board size 451 x 33 mm -> 461.5 x 33 mm

Commit message: update pcb
Parts:
- removed C108: 220n, Capacitor_SMD:C_0402_1005Metric
- removed the C501 at (453.7, 141.0)
- removed C502, C503: 0.1u, Capacitor_SMD:C_0402_1005Metric
- removed the R501 at (450.9, 141.0)
- removed U104: MS8607, clock:MS8607
- added Q501: BSS138, Package_TO_SOT_SMD:SOT-23, B.Cu at (452.3, 181.8)
- added R502: 10, Resistor_SMD:R_0402_1005Metric, B.Cu at (454.8, 181.3)
- C104, C114, C115, C116, C301, C302, C303, C304, C305, C306, C307, C308, C309, C310, C311, C312, C313, C314, C315, C316, C317, C318, C319, C320, C321, C322, C323, C324, C325, C326, C327, C328, C401, J101, L401, R101, R105, R106, R107, R108, R207, R301, R302, R303, R304, R305, R306, R307, R308, R309, R310, R311, R312, R313, R314, R401, SW101, U102, U303, U304, U307, U308, U311, U312, U317, U318, U320, U322, U324, U325, U329, U330, U333, U334, U338: moved to B.Cu
- C501: renamed from C504; value 10u -> 1u; moved to B.Cu
- J501: value 1-1734839-6 -> IPS_80x160_0.96; footprint clock:TE_1-1734839-6 -> clock:IPS_FPC-13
- R501: renamed from R502; value 5.1k -> 10k; moved to B.Cu
- SW102, SW103: footprint clock:EVQP4xB3x -> Button_Switch_SMD:SW_SPST_EVQP2; moved to F.Cu
- moved C303 301.5 mm to (54.3, 159.6), turned to 180 degrees
- moved R106 279.5 mm to (466.9, 175.2), turned to 180 degrees
- moved C302 268.2 mm to (54.7, 177.4)
- moved C304 260.2 mm to (54.7, 176.4)
- moved R105 256.4 mm to (451.1, 176.8), turned to 90 degrees
- moved J102 245.0 mm to (430.0, 165.4)
- moved SW101 243.2 mm to (429.7, 162.7), turned to 180 degrees
- moved R108 242.2 mm to (436.7, 165.0), turned to -90 degrees
- moved U102 242.0 mm to (437.5, 154.1)
- moved R107 241.3 mm to (438.3, 164.5)
- moved C307 239.9 mm to (122.3, 159.6), turned to 180 degrees
- moved C115 238.9 mm to (444.2, 175.8), turned to -90 degrees
- moved R101 238.3 mm to (450.5, 175.3), turned to 180 degrees
- moved C116 237.8 mm to (444.2, 165.4), turned to 90 degrees
- moved C114 236.4 mm to (448.4, 175.3)
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Connections:
- C501 pad 2: Net-(C504-Pad2) -> +3V3
- J501 pad 1: Net-(C502-Pad2) -> unconnected-(J501-Pad1)
- J501 pad 10: /OLED_D/C -> +3V3
- J501 pad 11: /OLED_SCK -> /Display/LED_K
- J501 pad 12: /OLED_MOSI -> +3V3
- J501 pad 13: Net-(J501-Pad13) -> Earth
- J501 pad 2: Net-(C502-Pad1) -> unconnected-(J501-Pad2)
- J501 pad 3: Net-(C503-Pad2) -> /DISP_COPI
- J501 pad 4: Earth -> /DISP_CLK
- J501 pad 5: Net-(C503-Pad1) -> /DISP_DC
- J501 pad 6: +3V3 -> /DISP_RST
- J501 pad 7: +3V3 -> /DISP_CS
- J501 pad 8: /OLED_CS -> Earth
- J501 pad 9: /OLED_RST -> unconnected-(J501-Pad9)
- R207 pad 1: /Power/SEG_2.5V_TOP_EN -> /SEG_2.5V_TOP_EN
- R208 pad 1: /Power/SEG_2.5V_BOT_EN -> /SEG_2.5V_BOT_EN
- R501 pad 1: Earth -> /DISP_BL
- R501 pad 2: /OLED_RST -> +3V3
- U103 pad 11: Net-(J102-Pad2) -> /DISP_BL
- U103 pad 12: Net-(J102-Pad1) -> /SEG_MOSI
- U103 pad 13: /GPS_TX -> /SEG_LAT
- U103 pad 14: /GPS_RX -> /SEG_CLK
- U103 pad 15: /GPS_PPS -> /SEG_OE
- U103 pad 16: unconnected-(U103-Pad16) -> Net-(J102-Pad2)
- U103 pad 17: unconnected-(U103-Pad17) -> Net-(J102-Pad1)
- U103 pad 18: unconnected-(U103-Pad18) -> /GPS_TX
- U103 pad 2: unconnected-(U103-Pad2) -> /POW_SDA
- U103 pad 27: /BTN_UP -> /GPS_RX
- U103 pad 28: /BTN_DWN -> /GPS_PPS
- U103 pad 29: /SEN_SCL -> unconnected-(U103-Pad29)
- U103 pad 3: unconnected-(U103-Pad3) -> /POW_SCL
- U103 pad 30: /SEN_SDA -> unconnected-(U103-Pad30)
- U103 pad 31: /OLED_MOSI -> unconnected-(U103-Pad31)
- U103 pad 32: /OLED_SCK -> unconnected-(U103-Pad32)
- U103 pad 34: /OLED_D/C -> /SEN_SCL
- U103 pad 35: /OLED_RST -> /SEN_SDA
- U103 pad 36: /OLED_CS -> /BTN_UP
- U103 pad 37: unconnected-(U103-Pad37) -> /BATT_EN
- U103 pad 38: /BATT_EN -> /SEG_2.5V_TOP_EN
- U103 pad 39: /POW_SCL -> /BC_INT
- U103 pad 4: unconnected-(U103-Pad4) -> /DISP_CS
- U103 pad 40: /POW_SDA -> /SEG_2.5V_BOT_EN
- U103 pad 5: unconnected-(U103-Pad5) -> /DISP_RST
- U103 pad 6: /SEG_MOSI -> /DISP_DC
- U103 pad 7: /SEG_LAT -> /DISP_CLK
- U103 pad 8: /SEG_CLK -> /DISP_COPI
- U103 pad 9: /SEG_OE -> /BTN_DWN
- U203 pad 7: /Power/BC_~{INT} -> /BC_INT
- U204 pad 1: /Power/SEG_2.5V_TOP_EN -> /SEG_2.5V_TOP_EN
- U205 pad 1: /Power/SEG_2.5V_BOT_EN -> /SEG_2.5V_BOT_EN
Routing:
- net /BTN_UP: track 0.00 -> 43.9 mm, vias 0 -> 3
- net /POW_SCL: track 0.00 -> 36.3 mm, vias 0 -> 2
- net /POW_SDA: track 0.00 -> 33.8 mm, vias 0 -> 2
- net /BTN_DWN: track 5.39 -> 36.5 mm, vias 2 -> 1
- net SEG_2.5V_BOT: track 5.48 -> 32.5 mm, vias 0 -> 10
- net /DISP_COPI: track 0.00 -> 25.1 mm
- net +3V3: track 26.3 -> 50.9 mm, vias 20 -> 32
- net Earth: track 46.2 -> 70.3 mm, vias 63 -> 83
- net /DISP_CLK: track 0.00 -> 23.7 mm
- net /DISP_DC: track 0.00 -> 22.2 mm
- net /SEN_SCL: track 0.00 -> 22.0 mm, vias 0 -> 2
- net /DISP_RST: track 0.00 -> 20.7 mm
- net /SEG_2.5V_BOT_EN: track 0.00 -> 20.2 mm, vias 0 -> 2
- net /SEN_SDA: track 0.00 -> 19.3 mm, vias 0 -> 2
- net /DISP_CS: track 0.00 -> 19.3 mm
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- added copper zone on B.Cu, net SEG_2.5V_BOT
- removed copper zone on In1.Cu, net +BATT
Other:
- board size 461.5 x 33 mm -> 462 x 33 mm

Commit message: update pcb
Parts:
- removed AE401: Active, Capacitor_SMD:C_0603_1608Metric
- removed J102: UART, Connector_PinHeader_1.27mm:PinHeader_1x02_P1.27mm_Vertical
- added BT201: Lipo, Connector_JST:JST_PH_S2B-PH-K_1x02_P2.00mm_Horizontal, B.Cu at (348.5, 163.6)
- added BT202: Lipo, Connector_JST:JST_PH_S2B-PH-K_1x02_P2.00mm_Horizontal, B.Cu at (238.0, 163.7)
- added BT203: Lipo, Connector_JST:JST_PH_S2B-PH-K_1x02_P2.00mm_Horizontal, B.Cu at (129.5, 163.6)
- added C329: 1u, Capacitor_SMD:C_0402_1005Metric, B.Cu at (120.9, 174.9)
- added C330: 1u, Capacitor_SMD:C_0402_1005Metric, B.Cu at (119.0, 161.1)
- added C331: 1u, Capacitor_SMD:C_0402_1005Metric, B.Cu at (229.3, 174.9)
- added C332: 1u, Capacitor_SMD:C_0402_1005Metric, B.Cu at (226.8, 161.1)
- added C333: 1u, Capacitor_SMD:C_0402_1005Metric, B.Cu at (336.3, 161.1)
- added C334: 1u, Capacitor_SMD:C_0402_1005Metric, B.Cu at (332.7, 174.9)
- added G***: LOGO, clock:satellite, B.Cu at (380.6, 164.3)
- added JP201: Jumper_2_Bridged, Connector_PinHeader_2.54mm:PinHeader_1x02_P2.54mm_Horizontal, B.Cu at (244.2, 166.5)
- added JP202: Jumper_2_Bridged, Connector_PinHeader_2.54mm:PinHeader_1x02_P2.54mm_Horizontal, B.Cu at (134.2, 166.5)
- added R217: 50, Resistor_SMD:R_1206_3216Metric, B.Cu at (245.5, 163.5)
- added R218: 50, Resistor_SMD:R_1206_3216Metric, B.Cu at (135.5, 163.5)
- added SW104: RUN, Button_Switch_SMD:SW_SPST_EVQP2, B.Cu at (425.1, 168.0)
- J101: value SWD -> Conn_01x07; footprint Connector_PinHeader_1.27mm:PinHeader_1x03_P1.27mm_Vertical -> Connector_PinHeader_1.27mm:PinHeader_1x07_P1.27mm_Vertical
- SW101: footprint clock:EVQP4xB3x -> Button_Switch_SMD:SW_SPST_EVQP2
- SW102: value SW_Push -> BTN_UP
- SW103: value SW_Push -> BTN_DWN
- moved U307 34.4 mm to (122.7, 174.9)
- moved U308 29.0 mm to (117.3, 161.1)
- moved C401 28.2 mm to (409.7, 170.9), turned to 180 degrees
- moved U401 27.5 mm to (417.0, 169.5)
- moved R401 27.2 mm to (410.2, 169.5)
- moved L401 27.2 mm to (410.2, 172.3)
- moved J401 27.1 mm to (407.2, 172.8)
- moved U320 20.0 mm to (231.0, 174.9)
- moved J101 18.2 mm to (435.3, 159.2), turned to 90 degrees
- moved U322 14.2 mm to (225.1, 161.1)
- moved SW101 5.27 mm to (429.9, 168.0), turned to 90 degrees
- moved U334 3.60 mm to (334.5, 174.9)
- moved U333 3.50 mm to (334.5, 161.1)
- moved C314 0.10 mm to (231.0, 177.4)
- moved C316 0.10 mm to (231.0, 176.4)
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Connections:
- J101 pad 1: /RUN -> +3V3
- J101 pad 2: /SWD -> /UART_TX
- J101 pad 3: /SWCLK -> /UART_RX
- U103 pad 12: /SEG_MOSI -> /SEG_LAT
- U103 pad 13: /SEG_LAT -> /SEG_CLK
- U103 pad 14: /SEG_CLK -> /SEG_MOSI
- U103 pad 16: Net-(J102-Pad2) -> unconnected-(U103-Pad16)
- U103 pad 17: Net-(J102-Pad1) -> unconnected-(U103-Pad17)
- U103 pad 18: /GPS_TX -> unconnected-(U103-Pad18)
- U103 pad 27: /GPS_RX -> /GPS_PPS
- U103 pad 28: /GPS_PPS -> /GPS_RX
- U103 pad 29: unconnected-(U103-Pad29) -> /GPS_TX
- U103 pad 30: unconnected-(U103-Pad30) -> /UART_RX
- U103 pad 31: unconnected-(U103-Pad31) -> /UART_TX
- U303 pad 10: /Segments/DG0_A -> /Segments/DG0_B
- U303 pad 11: /Segments/DG0_B -> /Segments/DG0_A
- U303 pad 14: /Segments/DG1_A -> /Segments/DG1_B
- U303 pad 15: /Segments/DG1_B -> /Segments/DG1_A
- U303 pad 18: /Segments/DG2_A -> /Segments/DG2_B
- U303 pad 19: /Segments/DG2_B -> /Segments/DG2_A
- U303 pad 22: /Segments/DG3_A -> /Segments/DG3_B
- U303 pad 23: /Segments/DG3_B -> /Segments/DG3_A
- U304 pad 10: /Segments/DG3_D -> /Segments/DG3_E
- U304 pad 11: /Segments/DG3_E -> /Segments/DG3_D
- U304 pad 14: /Segments/DG2_D -> /Segments/DG2_E
- U304 pad 15: /Segments/DG2_E -> /Segments/DG2_D
- U304 pad 18: /Segments/DG1_D -> /Segments/DG1_E
- U304 pad 19: /Segments/DG1_E -> /Segments/DG1_D
- U304 pad 22: /Segments/DG0_D -> /Segments/DG0_E
- U304 pad 23: /Segments/DG0_E -> /Segments/DG0_D
- U311 pad 10: /Segments/DG4_A -> /Segments/DG4_B
- U311 pad 11: /Segments/DG4_B -> /Segments/DG4_A
- U311 pad 14: /Segments/DG5_A -> /Segments/DG5_B
- U311 pad 15: /Segments/DG5_B -> /Segments/DG5_A
- U311 pad 18: /Segments/DG6_A -> /Segments/DG6_B
- U311 pad 19: /Segments/DG6_B -> /Segments/DG6_A
- U311 pad 22: /Segments/DG7_A -> /Segments/DG7_B
- U311 pad 23: /Segments/DG7_B -> /Segments/DG7_A
- U312 pad 10: /Segments/DG7_D -> /Segments/DG7_E
- U312 pad 11: /Segments/DG7_E -> /Segments/DG7_D
- U312 pad 14: /Segments/DG6_D -> /Segments/DG6_E
- U312 pad 15: /Segments/DG6_E -> /Segments/DG6_D
- U312 pad 18: /Segments/DG5_D -> /Segments/DG5_E
- U312 pad 19: /Segments/DG5_E -> /Segments/DG5_D
- U312 pad 22: /Segments/DG4_D -> /Segments/DG4_E
- U312 pad 23: /Segments/DG4_E -> /Segments/DG4_D
- U317 pad 10: /Segments/DG8_A -> /Segments/DG8_B
- U317 pad 11: /Segments/DG8_B -> /Segments/DG8_A
- U317 pad 14: /Segments/DG9_A -> /Segments/DG9_B
- U317 pad 15: /Segments/DG9_B -> /Segments/DG9_A
- U318 pad 18: /Segments/DG9_D -> /Segments/DG9_E
- U318 pad 19: /Segments/DG9_E -> /Segments/DG9_D
- U318 pad 22: /Segments/DG8_D -> /Segments/DG8_E
- U318 pad 23: /Segments/DG8_E -> /Segments/DG8_D
- U324 pad 10: /Segments/DG11_A -> /Segments/DG11_B
- U324 pad 11: /Segments/DG11_B -> /Segments/DG11_A
- U324 pad 14: /Segments/DG12_A -> /Segments/DG12_B
- U324 pad 15: /Segments/DG12_B -> /Segments/DG12_A
- U324 pad 16: /Segments/COL0_T -> unconnected-(U324-Pad16)
- U324 pad 17: unconnected-(U324-Pad17) -> /Segments/DG13_G
- U324 pad 18: /Segments/DG13_G -> /Segments/DG13_F
- U324 pad 19: /Segments/DG13_F -> /Segments/DG13_B
- U324 pad 21: /Segments/DG13_B -> /Segments/DG14_G
- U324 pad 22: /Segments/DG14_G -> /Segments/DG14_F
- U324 pad 23: /Segments/DG14_F -> /Segments/COL0_T
- U325 pad 10: /Segments/DG13_DP -> /Segments/DG14_D
- U325 pad 11: /Segments/DG13_C -> /Segments/DG13_DP
- U325 pad 12: /Segments/DG13_D -> /Segments/DG13_C
- U325 pad 14: /Segments/COL0_B -> /Segments/DG13_D
- U325 pad 18: /Segments/DG12_D -> /Segments/DG12_E
- U325 pad 19: /Segments/DG12_E -> /Segments/DG12_D
- U325 pad 22: /Segments/DG11_D -> /Segments/DG11_E
- U325 pad 23: /Segments/DG11_E -> /Segments/DG11_D
- U325 pad 8: /Segments/DG14_D -> /Segments/COL0_B
- U329 pad 10: /Segments/DG14_B -> /Segments/DG14_A
- U329 pad 13: /Segments/DG15_A -> /Segments/DG15_B
- U329 pad 14: /Segments/DG15_B -> /Segments/DG15_A
- U329 pad 17: /Segments/DG16_A -> /Segments/DG16_B
- U329 pad 18: /Segments/DG16_B -> /Segments/DG16_A
- U329 pad 21: /Segments/DG17_A -> /Segments/DG17_B
- U329 pad 22: /Segments/DG17_B -> /Segments/DG17_A
- U329 pad 9: /Segments/DG14_A -> /Segments/DG14_B
- U330 pad 11: /Segments/DG17_D -> /Segments/DG17_E
- U330 pad 12: /Segments/DG17_E -> /Segments/DG17_D
- U330 pad 15: /Segments/DG16_D -> /Segments/DG16_E
- U330 pad 16: /Segments/DG16_E -> /Segments/DG16_D
- U330 pad 19: /Segments/DG15_D -> /Segments/DG15_E
- U330 pad 20: /Segments/DG15_E -> /Segments/DG15_D
- U330 pad 21: /Segments/COL1_B -> /Segments/DG14_DP
- U330 pad 22: /Segments/DG14_DP -> /Segments/DG14_C
- U330 pad 23: /Segments/DG14_C -> /Segments/COL1_B
- U330 pad 8: /Segments/DG18_E -> /Segments/DG18_D
- U337 pad 10: /Segments/DG18_B -> /Segments/DG18_A
- U337 pad 13: /Segments/DG19_A -> /Segments/DG19_B
- U337 pad 14: /Segments/DG19_B -> /Segments/DG19_A
- U337 pad 15: /Segments/DG20_F -> unconnected-(U337-Pad15)
- U337 pad 16: /Segments/DG20_G -> /Segments/DG20_F
- U337 pad 17: /Segments/DG20_H -> /Segments/DG20_G
- U337 pad 18: unconnected-(U337-Pad18) -> /Segments/DG20_H
- U337 pad 20: /Segments/DG20_J -> /Segments/DG20_A
- U337 pad 21: /Segments/DG20_K -> /Segments/DG20_J
- U337 pad 23: /Segments/DG20_A -> /Segments/DG20_K
- U337 pad 9: /Segments/DG18_A -> /Segments/DG18_B
- U338 pad 10: /Segments/DG20_C -> /Segments/DG20_L
- U338 pad 11: /Segments/DG20_L -> /Segments/DG20_M
- U338 pad 12: /Segments/DG20_M -> /Segments/DG21_D
- U338 pad 19: /Segments/DG19_D -> /Segments/DG19_E
- U338 pad 20: /Segments/DG19_E -> /Segments/DG19_D
- U338 pad 23: /Segments/DG18_D -> /Segments/DG18_E
- U338 pad 8: /Segments/DG21_D -> /Segments/DG20_DP
- U338 pad 9: /Segments/DG20_DP -> /Segments/DG20_C
Routing:
- net /Segments/SEG_LAT_BF2: track 0.00 -> 160.4 mm, vias 0 -> 5
- net /Segments/SEG_CLK_BF2: track 0.00 -> 155.9 mm, vias 0 -> 5
- net /SEG_LAT: track 0.00 -> 126.4 mm, vias 0 -> 4
- net /SEG_CLK: track 0.00 -> 122.1 mm, vias 0 -> 4
- net /Segments/SEG_LAT_BF1: track 0.00 -> 121.5 mm, vias 0 -> 4
- net /Segments/SEG_LAT_BF4: track 0.00 -> 118.5 mm, vias 0 -> 4
- net /Segments/SEG_CLK_BF4: track 0.00 -> 118.1 mm, vias 0 -> 4
- net /Segments/SEG_CLK_BF3: track 0.00 -> 116.8 mm, vias 0 -> 4
- net /Segments/SEG_LAT_BF3: track 0.00 -> 116.7 mm, vias 0 -> 4
- net /Segments/SEG_CLK_BF1: track 0.00 -> 116.7 mm, vias 0 -> 4
- net /Segments/SEG_CLK_BF0: track 0.00 -> 112.1 mm, vias 0 -> 4
- net /Segments/SEG_LAT_BF0: track 0.00 -> 111.9 mm, vias 0 -> 4
- net /Segments/SEG_CLK_BF5: track 0.00 -> 88.2 mm, vias 0 -> 4
- net /Segments/SEG_LAT_BF5: track 0.00 -> 87.5 mm, vias 0 -> 4
- net Earth: track 70.3 -> 149.6 mm, vias 83 -> 210
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- added copper zone on B.Cu, net Net-(BT202-Pad1)
- added copper zone on B.Cu, net Net-(BT203-Pad1)
Other:
- board text added: "3V3"
- board text added: "BOOT_SEL"
- board text added: "CLK"
- board text added: "GND"
- board text added: "GPS_CLock"
- board text added: "RESET"
- board text added: "RUN"
- board text added: "SWD"
- board text added: "UART_RX"
- board text added: "UART_TX"
- board text added: "USB PD 3.0: 5V/3A 9V/2A"
- board text added: "V1.0 2023-01"
