File: kicad/GPS_CLock/GPS_CLock.kicad_pcb (KiCad board)
At the start: 4 copper layers, 462 x 33 mm, 204 parts, among them J101 Conn_01x07, J201 USB_C_2.0, J401 U.FL, J501 IPS_80x160_0.96, Q201 PMPB17EP, Q202 PMPB17EP, Q501 BSS138, SW101 BOOT_JMP, SW102 BTN_UP, SW103 BTN_DWN, SW104 RUN, U101 W25Q16JVUXIQ, U102 VEML7700-TR, U103 RP2040, U201 LP5912-3.3DRV, U202 STUSB4500QTR, U203 BQ25892, U204 TPS62827DMQ, U205 TPS62827DMQ, U301 DG0, U302 DG1, U303 LED_CC7, U304 LED_CC6, U305 DG2, U306 DG3, U307 74AUP2G17, U308 74AUP2G17, U309 DG4, U310 DG5, U311 LED_CC8, U312 LED_CC5, U313 DG6, U314 DG7, U315 DG8, U316 DG9, U317 LED_CC9, U318 LED_CC4, U319 DG10, U320 74AUP2G17, U321 DG11, U322 74AUP2G17, U323 DG12, U324 LED_CC10, U325 LED_CC3, U326 DG13, U327 DG14, U328 DG15, U329 LED_CC11, U330 LED_CC2, U331 DG16, U332 DG17, U333 74AUP2G17, U334 74AUP2G17, U335 DG18, U336 DG19, U337 LED_CC12, U338 LED_CC1, U339 DG20, U340 DG21, U341 DG22, U342 LED_CC13, U343 LED_CC0, U344 DG23, U345 DG24, U401 MAX-M10S

Commit message: update pcb
Parts:
- added C335: 1u, Capacitor_SMD:C_0402_1005Metric, B.Cu at (157.8, 168.6)
- added C336: 1u, Capacitor_SMD:C_0402_1005Metric, B.Cu at (285.1, 168.6)
- added C337: 1u, Capacitor_SMD:C_0402_1005Metric, B.Cu at (388.0, 175.6)
- added U346: 74AUP2G17, clock:XSON-6_SOT886, B.Cu at (159.5, 168.5)
- added U347: 74AUP2G17, clock:XSON-6_SOT886, B.Cu at (286.8, 168.5)
- added U348: 74AUP2G17, clock:XSON-6_SOT886, B.Cu at (389.7, 175.5)
- SW101, SW102, SW103, SW104: footprint Button_Switch_SMD:SW_SPST_EVQP2 -> clock:SW_SPST_EVQP2
- moved C101 5.00 mm to (443.1, 173.7)
- moved C102 5.00 mm to (443.1, 171.7)
- moved C103 5.00 mm to (457.6, 175.3)
- moved C104 5.00 mm to (442.4, 155.3)
- moved C105 5.00 mm to (444.6, 169.2)
- moved C106 5.00 mm to (455.4, 171.3)
- moved C107 5.00 mm to (455.4, 168.8)
- moved C109 5.00 mm to (455.4, 167.9)
- moved C110 5.00 mm to (455.4, 166.9)
- moved C111 5.00 mm to (455.4, 170.3)
- moved C112 5.00 mm to (453.4, 165.8)
- moved C113 5.00 mm to (444.6, 170.2)
- moved C114 5.00 mm to (453.4, 175.3)
- moved C115 5.00 mm to (449.2, 175.8)
- moved C116 5.00 mm to (449.2, 165.4)
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Connections:
- U103 pad 16: unconnected-(U103-Pad16) -> /PD_INT
- U202 pad 19: unconnected-(U202-Pad19) -> /PD_INT
- U303 pad 24: /SEG_OE -> /Segments/SEG_OE_BF2
- U304 pad 24: /SEG_OE -> /Segments/SEG_OE_BF2
- U311 pad 24: /SEG_OE -> /Segments/SEG_OE_BF2
- U312 pad 24: /SEG_OE -> /Segments/SEG_OE_BF2
- U317 pad 24: /SEG_OE -> /Segments/SEG_OE_BF1
- U318 pad 24: /SEG_OE -> /Segments/SEG_OE_BF1
- U324 pad 24: /SEG_OE -> /Segments/SEG_OE_BF1
- U325 pad 24: /SEG_OE -> /Segments/SEG_OE_BF1
- U329 pad 24: /SEG_OE -> /Segments/SEG_OE_BF0
- U330 pad 24: /SEG_OE -> /Segments/SEG_OE_BF0
- U337 pad 24: /SEG_OE -> /Segments/SEG_OE_BF0
- U338 pad 24: /SEG_OE -> /Segments/SEG_OE_BF0
Routing:
- net /Segments/SEG_OE_BF1: track 0.00 -> 179.3 mm, vias 0 -> 8
- net /Segments/SEG_OE_BF0: track 0.00 -> 158.6 mm, vias 0 -> 8
- net /Segments/SEG_OE_BF2: track 0.00 -> 154.3 mm, vias 0 -> 8
- net /SEG_OE: track 0.00 -> 87.6 mm, vias 0 -> 4
- net /PD_INT: track 0.00 -> 30.2 mm, vias 0 -> 2
- net Earth: track 149.6 -> 153.4 mm, vias 210 -> 216
- net +3V3: track 92.2 -> 95.1 mm, vias 69 -> 72
- net /Segments/SEG_LAT_BF5: track 87.5 -> 88.5 mm
- net /Segments/SEG_LAT_BF3: track 116.7 -> 117.7 mm
- net /Segments/SEG_LAT_BF1: track 121.5 -> 122.5 mm
- net /Segments/SEG_CLK_BF5: track 88.2 -> 89.2 mm
- net /Segments/SEG_CLK_BF3: track 116.8 -> 117.8 mm
- net /Segments/SEG_CLK_BF1: track 116.7 -> 117.7 mm
- net /SEG_LAT: track 126.4 -> 127.4 mm
- net /SEG_CLK: track 122.1 -> 123.1 mm
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Other:
- board size 462 x 33 mm -> 464 x 33 mm
- board text added: "A0"
- board text added: "A1"
- board text added: "C0"
- board text added: "C1"
- board text added: "C2"
- board text added: "N0"
- board text added: "N1"
- board text added: "N10"
- board text added: "N11"
- board text added: "N12"
- board text added: "N13"
- board text added: "N14"
- board text added: "N15"
- board text added: "N16"
- board text added: "N17"
- board text added: "N18"
- board text added: "N19"
- board text added: "N2"
- board text added: "N20"
- board text added: "N21"
- board text added: "N22"
- board text added: "N3"
- board text added: "N4"
- board text added: "N5"
- board text added: "N6"
- board text added: "N7"
- board text added: "N8"
- board text added: "N9"
- board text added: "USB PD INPUT: 5V/3A 9V/1.67A 12V/1.25A"
- board text removed: "USB PD 3.0: 5V/3A 9V/2A"
