File: kicad/GPS_CLock/Segments.kicad_sch (KiCad schematic)
At the start: 89 parts, among them U301 DG0, U302 DG1, U303 LED_CC7, U304 LED_CC6, U305 DG2, U306 DG3, U307 DG4, U308 DG5, U309 LED_CC8, U310 LED_CC5, U311 DG6, U312 DG7, U313 DG8, U314 DG9, U315 LED_CC9, U316 LED_CC4, U317 DG10, U318 DG11, U319 DG12, U320 LED_CC10, U321 LED_CC3, U322 DG13, U323 DG14, U324 DG15, U325 LED_CC11, U326 LED_CC2, U327 DG16, U328 DG17, U329 DG18, U330 DG19, U331 LED_CC12, U332 LED_CC1, U333 DG20, U334 DG21, U335 DG22, U336 LED_CC13, U337 LED_CC0, U338 DG23, U339 DG24, U340 74LVC3G17

Commit message: change to larger segments
Parts:
- removed C329: 0.1u, Capacitor_SMD:C_0402_1005Metric, symbol Device:C_Small
- removed U340: 74LVC3G17, clock:PSON50P100X195X50-8N, symbol Clock:74LVC3G17
- added U307, U308, U320, U322, U333, U334: 74AUP2G17, clock:XSON-6_SOT886, symbol Clock:74AUP2G17
- U301, U302, U305, U306: footprint clock:7seg 0.56in smd -> clock:7seg 0.8in smd; symbol Clock:7-SegmentLED -> Clock:7-SegmentLED_0.8_SMD
- U309: renamed from U307; footprint clock:7seg 0.56in smd -> clock:7seg 0.8in smd; symbol Clock:7-SegmentLED -> Clock:7-SegmentLED_0.8_SMD
- U310: renamed from U308; footprint clock:7seg 0.56in smd -> clock:7seg 0.8in smd; symbol Clock:7-SegmentLED -> Clock:7-SegmentLED_0.8_SMD
- U313: renamed from U311; footprint clock:7seg 0.56in smd -> clock:7seg 0.8in smd; symbol Clock:7-SegmentLED -> Clock:7-SegmentLED_0.8_SMD
- U314: renamed from U312; footprint clock:7seg 0.56in smd -> clock:7seg 0.8in smd; symbol Clock:7-SegmentLED -> Clock:7-SegmentLED_0.8_SMD
- U315: renamed from U313; footprint clock:7seg 0.56in smd -> clock:7seg 0.8in smd; symbol Clock:7-SegmentLED -> Clock:7-SegmentLED_0.8_SMD
- U316: renamed from U314; footprint clock:7seg 0.56in smd -> clock:7seg 0.8in smd; symbol Clock:7-SegmentLED -> Clock:7-SegmentLED_0.8_SMD
- U321: renamed from U318; footprint clock:7seg 0.56in smd -> clock:7seg 0.8in smd; symbol Clock:7-SegmentLED -> Clock:7-SegmentLED_0.8_SMD
- U323: renamed from U319; footprint clock:7seg 0.56in smd -> clock:7seg 0.8in smd; symbol Clock:7-SegmentLED -> Clock:7-SegmentLED_0.8_SMD
- U326: renamed from U322; footprint clock:7seg 0.56in smd -> clock:7seg 0.8in smd; symbol Clock:7-SegmentLED -> Clock:7-SegmentLED_0.8_SMD
- U327: renamed from U323; footprint clock:7seg 0.56in smd -> clock:7seg 0.8in smd; symbol Clock:7-SegmentLED -> Clock:7-SegmentLED_0.8_SMD
- U328: renamed from U324; footprint clock:7seg 0.56in smd -> clock:7seg 0.8in smd; symbol Clock:7-SegmentLED -> Clock:7-SegmentLED_0.8_SMD
- U331: renamed from U327; footprint clock:7seg 0.56in smd -> clock:7seg 0.8in smd; symbol Clock:7-SegmentLED -> Clock:7-SegmentLED_0.8_SMD
- U332: renamed from U328; footprint clock:7seg 0.56in smd -> clock:7seg 0.8in smd; symbol Clock:7-SegmentLED -> Clock:7-SegmentLED_0.8_SMD
- U335: renamed from U329; footprint clock:7seg 0.56in smd -> clock:7seg 0.8in smd; symbol Clock:7-SegmentLED -> Clock:7-SegmentLED_0.8_SMD
- U336: renamed from U330; footprint clock:7seg 0.56in smd -> clock:7seg 0.8in smd; symbol Clock:7-SegmentLED -> Clock:7-SegmentLED_0.8_SMD
- U340: renamed from U334; footprint clock:7seg 0.56in smd -> clock:7seg 0.8in smd; symbol Clock:7-SegmentLED -> Clock:7-SegmentLED_0.8_SMD
- U341: renamed from U335; footprint clock:7seg 0.56in smd -> clock:7seg 0.8in smd; symbol Clock:7-SegmentLED -> Clock:7-SegmentLED_0.8_SMD
- U344: renamed from U338; footprint clock:7seg 0.56in smd -> clock:7seg 0.8in smd; symbol Clock:7-SegmentLED -> Clock:7-SegmentLED_0.8_SMD
- U345: renamed from U339; footprint clock:7seg 0.56in smd -> clock:7seg 0.8in smd; symbol Clock:7-SegmentLED -> Clock:7-SegmentLED_0.8_SMD
- renumbered U309 to U311, U310 to U312, U315 to U317, U316 to U318, U317 to U319, U320 to U324, U321 to U325, U325 to U329, U326 to U330, U331 to U337, U332 to U338, U333 to U339, U336 to U342, U337 to U343
Connections:
- net LED_OE_BF0 is gone; now on net SEG_OE_CONN: U325.24 (OE), U330.24 (OE)
- net +3V3: now also U307.5 (VDD), U308.5 (VDD), U320.5 (VDD), U322.5 (VDD), U333.5 (VDD), U334.5 (VDD)
- net DG0_B: now also U301.8 (B); no longer U301.6 (B)
- net DG0_E: now also U301.3 (E); no longer U301.1 (E)
- net DG11_B: now also U321.8 (B); no longer U321.6 (B)
- net DG11_E: now also U321.3 (E); no longer U321.1 (E)
- net DG12_B: now also U323.8 (B); no longer U323.6 (B)
- net DG12_E: now also U323.3 (E); no longer U323.1 (E)
- net DG13_B: now also U326.8 (B); no longer U326.6 (B)
- net DG13_E: now also U326.3 (E); no longer U326.1 (E)
- net DG14_B: now also U327.8 (B); no longer U327.6 (B)
- net DG14_E: now also U327.3 (E); no longer U327.1 (E)
- net DG15_B: now also U328.8 (B); no longer U328.6 (B)
- net DG15_E: now also U328.3 (E); no longer U328.1 (E)
- net DG16_B: now also U331.8 (B); no longer U331.6 (B)
- net DG16_E: now also U331.3 (E); no longer U331.1 (E)
- net DG17_B: now also U332.8 (B); no longer U332.6 (B)
- net DG17_E: now also U332.3 (E); no longer U332.1 (E)
- net DG18_B: now also U335.8 (B); no longer U335.6 (B)
- net DG18_E: now also U335.3 (E); no longer U335.1 (E)
- net DG19_B: now also U336.8 (B); no longer U336.6 (B)
- net DG19_E: now also U336.3 (E); no longer U336.1 (E)
- net DG1_B: now also U302.8 (B); no longer U302.6 (B)
- net DG1_E: now also U302.3 (E); no longer U302.1 (E)
- net DG21_B: now also U340.8 (B); no longer U340.6 (B)
- net DG21_E: now also U340.3 (E); no longer U340.1 (E)
- net DG22_B: now also U341.8 (B); no longer U341.6 (B)
- net DG22_E: now also U341.3 (E); no longer U341.1 (E)
- net DG23_B: now also U344.8 (B); no longer U344.6 (B)
- net DG23_E: now also U344.3 (E); no longer U344.1 (E)
- net DG24_B: now also U345.8 (B); no longer U345.6 (B)
- net DG24_E: now also U345.3 (E); no longer U345.1 (E)
- net DG2_B: now also U305.8 (B); no longer U305.6 (B)
- net DG2_E: now also U305.3 (E); no longer U305.1 (E)
- net DG3_B: now also U306.8 (B); no longer U306.6 (B)
- net DG3_E: now also U306.3 (E); no longer U306.1 (E)
- net DG4_B: now also U309.8 (B); no longer U309.6 (B)
- net DG4_E: now also U309.3 (E); no longer U309.1 (E)
- net DG5_B: now also U310.8 (B); no longer U310.6 (B)
- net DG5_E: now also U310.3 (E); no longer U310.1 (E)
- net DG6_B: now also U313.8 (B); no longer U313.6 (B)
- net DG6_E: now also U313.3 (E); no longer U313.1 (E)
- net DG7_B: now also U314.8 (B); no longer U314.6 (B)
- net DG7_E: now also U314.3 (E); no longer U314.1 (E)
- net DG8_B: now also U315.8 (B); no longer U315.6 (B)
- net DG8_E: now also U315.3 (E); no longer U315.1 (E)
- net DG9_B: now also U316.8 (B); no longer U316.6 (B)
- net DG9_E: now also U316.3 (E); no longer U316.1 (E)
- net Earth: now also U307.2 (GND), U308.2 (GND), U320.2 (GND), U322.2 (GND), U333.2 (GND), U334.2 (GND)
- net SEG_SOUT_CC10: now reaches U324.1 (SOUT)
- net SEG_SOUT_CC10: now also U329.5 (SIN)
- net SEG_SOUT_CC9: now reaches U324.5 (SIN)
- net SEG_SOUT_CC9: now also U317.1 (SOUT)
- net SEG_SOUT_CC11: now reaches U329.1 (SOUT)
- net SEG_SOUT_CC11: now also U337.5 (SIN)
- net SEG_SOUT_CC8: now reaches U317.5 (SIN)
- net SEG_SOUT_CC8: now also U311.1 (SOUT)
- net SEG_SOUT_CC12: now reaches U337.1 (SOUT)
- net SEG_SOUT_CC12: now also U342.5 (SIN)
- removed net +2V5: D301.2 (A), D302.2 (A), D303.2 (A), D304.2 (A), D305.2 (A), D306.2 (A), U301.3 (CA), U301.8 (CA), U302.3 (CA), U302.8 (CA), U305.3 (CA), U305.8 (CA), U306.3 (CA), U306.8 (CA), U309.3 (CA), U309.8 (CA), U310.3 (CA), U310.8 (CA), U313.3 (CA), U313.8 (CA), U314.3 (CA), U314.8 (CA), U315.3 (CA), U315.8 (CA), U316.3 (CA), U316.8 (CA), U319.14 (CA), U321.3 (CA), U321.8 (CA), U323.3 (CA), U323.8 (CA), U326.3 (CA), U326.8 (CA), U327.3 (CA), U327.8 (CA), U328.3 (CA), U328.8 (CA), U331.3 (CA), U331.8 (CA), U332.3 (CA), U332.8 (CA), U335.3 (CA), U335.8 (CA), U336.3 (CA), U336.8 (CA), U339.14 (CA), U340.3 (CA), U340.8 (CA), U341.3 (CA), U341.8 (CA), U344.3 (CA), U344.8 (CA), U345.3 (CA), U345.8 (CA)
- net CC0_CC1 renamed SEG_SOUT_CC0
- net CC1_CC2 renamed SEG_SOUT_CC1
- net CC2_CC3 renamed SEG_SOUT_CC2
- net CC3_CC4 renamed SEG_SOUT_CC3
- net CC4_CC5 renamed SEG_SOUT_CC4
- net CC5_CC6 renamed SEG_SOUT_CC5
- net CC6_CC7 renamed SEG_SOUT_CC6
- net CC7_CC8 renamed SEG_SOUT_CC7
- net SEG_SOUT_CC7: no longer U311.1 (SOUT)
- removed net LED_LAT: U303.7 (LAT), U304.7 (LAT), U311.7 (LAT), U312.7 (LAT), U317.7 (LAT), U318.7 (LAT), U324.7 (LAT), U329.7 (LAT), U337.7 (LAT), U338.7 (LAT), U342.7 (LAT), U343.7 (LAT)
- net LED_LAT_BF0 renamed SEG_LAT_BF0
- net SEG_LAT_BF0: now also U320.3 (2A), U334.4 (2Y)
- net LED_MOSI renamed SEG_SOUT_CONN
- net LED_OE renamed SEG_OE_CONN
- removed net LED_SCK: U303.6 (CLK), U304.6 (CLK), U311.6 (CLK), U312.6 (CLK), U317.6 (CLK), U318.6 (CLK), U324.6 (CLK), U329.6 (CLK), U337.6 (CLK), U338.6 (CLK), U342.6 (CLK), U343.6 (CLK)
- net LED_SCK_BF0 renamed SEG_CLK_BF0
- net SEG_CLK_BF0: now also U320.1 (1A), U334.6 (1Y)
- new net SEG_2.5V_BOT: D301.2 (A), D302.2 (A), D303.2 (A), D304.2 (A), D305.2 (A), D306.2 (A), U301.1 (CA), U302.1 (CA), U305.1 (CA), U306.1 (CA), U309.1 (CA), U310.1 (CA), U313.1 (CA), U314.1 (CA), U315.1 (CA), U316.1 (CA), U321.1 (CA), U323.1 (CA), U326.1 (CA), U327.1 (CA), U328.1 (CA), U331.1 (CA), U332.1 (CA), U335.1 (CA), U336.1 (CA), U340.1 (CA), U341.1 (CA), U344.1 (CA), U345.1 (CA)
- new net SEG_2.5V_TOP: U301.6 (CA), U302.6 (CA), U305.6 (CA), U306.6 (CA), U309.6 (CA), U310.6 (CA), U313.6 (CA), U314.6 (CA), U315.6 (CA), U316.6 (CA), U319.14 (CA), U321.6 (CA), U323.6 (CA), U326.6 (CA), U327.6 (CA), U328.6 (CA), U331.6 (CA), U332.6 (CA), U335.6 (CA), U336.6 (CA), U339.14 (CA), U340.6 (CA), U341.6 (CA), U344.6 (CA), U345.6 (CA)
- new net SEG_CLK_BF1: U307.1 (1A), U312.6 (CLK), U318.6 (CLK), U320.6 (1Y)
- new net SEG_CLK_BF2: U303.6 (CLK), U304.6 (CLK), U307.6 (1Y), U308.1 (1A)
- new net SEG_CLK_BF3: U308.6 (1Y), U311.6 (CLK), U317.6 (CLK), U322.1 (1A)
- new net SEG_CLK_BF4: U322.6 (1Y), U324.6 (CLK), U329.6 (CLK), U333.1 (1A)
- new net SEG_CLK_BF5: U333.6 (1Y), U337.6 (CLK), U342.6 (CLK)
- new net SEG_CLK_CONN: U334.1 (1A), U338.6 (CLK), U343.6 (CLK)
- new net SEG_LAT_BF1: U307.3 (2A), U312.7 (LAT), U318.7 (LAT), U320.4 (2Y)
- new net SEG_LAT_BF2: U303.7 (LAT), U304.7 (LAT), U307.4 (2Y), U308.3 (2A)
- new net SEG_LAT_BF3: U308.4 (2Y), U311.7 (LAT), U317.7 (LAT), U322.3 (2A)
- new net SEG_LAT_BF4: U322.4 (2Y), U324.7 (LAT), U329.7 (LAT), U333.3 (2A)
- new net SEG_LAT_BF5: U333.4 (2Y), U337.7 (LAT), U342.7 (LAT)
- new net SEG_LAT_CONN: U334.3 (2A), U338.7 (LAT), U343.7 (LAT)
- no-connect marks 1 -> 5

Commit message: updated pcb
Connections:
- net COL2_B: now also U343.23 (OUT15); no longer U343.16 (OUT8)
- net COL2_T: now also U342.8 (OUT0); no longer U342.23 (OUT15)
- net DG21_A: now also U342.11 (OUT3); no longer U342.9 (OUT1)
- net DG21_C: now also U343.21 (OUT13); no longer U343.22 (OUT14)
- net DG21_D: now also U338.8 (OUT0); no longer U343.23 (OUT15)
- net DG21_DP: now also U343.20 (OUT12); no longer U343.21 (OUT13)
- net DG21_E: now also U343.22 (OUT14); no longer U338.8 (OUT0)
- net DG21_F: now also U342.9 (OUT1); no longer U342.8 (OUT0)
- net DG22_A: now also U342.15 (OUT7); no longer U342.13 (OUT5)
- net DG22_C: now also U343.17 (OUT9); no longer U343.18 (OUT10)
- net DG22_DP: now also U343.16 (OUT8); no longer U343.17 (OUT9)
- net DG22_E: now also U343.18 (OUT10); no longer U343.20 (OUT12)
- net DG22_F: now also U342.13 (OUT5); no longer U342.12 (OUT4)
- net DG22_G: now also U342.12 (OUT4); no longer U342.11 (OUT3)
- net DG23_A: now also U342.19 (OUT11); no longer U342.17 (OUT9)
- net DG23_D: now also U343.15 (OUT7); no longer U343.14 (OUT6)
- net DG23_E: now also U343.14 (OUT6); no longer U343.15 (OUT7)
- net DG23_F: now also U342.17 (OUT9); no longer U342.16 (OUT8)
- net DG23_G: now also U342.16 (OUT8); no longer U342.15 (OUT7)
- net DG24_A: now also U342.23 (OUT15); no longer U342.21 (OUT13)
- net DG24_D: now also U343.11 (OUT3); no longer U343.10 (OUT2)
- net DG24_E: now also U343.10 (OUT2); no longer U343.11 (OUT3)
- net DG24_F: now also U342.21 (OUT13); no longer U342.20 (OUT12)
- net DG24_G: now also U342.20 (OUT12); no longer U342.19 (OUT11)
- net SEG_CLK_CONN renamed SEG_CLK_MCU
- net SEG_LAT_CONN renamed SEG_LAT_MCU
- net SEG_OE_CONN renamed SEG_OE_MCU
- net SEG_SOUT_CONN renamed SEG_SOUT_MCU

Commit message: update pcb
Parts:
- added C329, C330, C331, C332, C333, C334: 1u, Capacitor_SMD:C_0402_1005Metric, symbol Device:C_Small
Connections:
- net +3V3: now also C329.2, C330.2, C331.2, C332.2, C333.2, C334.2
- net COL0_B: now also U325.8 (OUT0); no longer U325.14 (OUT6)
- net COL0_T: now also U324.23 (OUT15); no longer U324.16 (OUT8)
- net COL1_B: now also U330.23 (OUT15); no longer U330.21 (OUT13)
- net DG0_A: now also U303.11 (OUT3); no longer U303.10 (OUT2)
- net DG0_B: now also U303.10 (OUT2); no longer U303.11 (OUT3)
- net DG0_D: now also U304.23 (OUT15); no longer U304.22 (OUT14)
- net DG0_E: now also U304.22 (OUT14); no longer U304.23 (OUT15)
- net DG11_A: now also U324.11 (OUT3); no longer U324.10 (OUT2)
- net DG11_B: now also U324.10 (OUT2); no longer U324.11 (OUT3)
- net DG11_D: now also U325.23 (OUT15); no longer U325.22 (OUT14)
- net DG11_E: now also U325.22 (OUT14); no longer U325.23 (OUT15)
- net DG12_A: now also U324.15 (OUT7); no longer U324.14 (OUT6)
- net DG12_B: now also U324.14 (OUT6); no longer U324.15 (OUT7)
- net DG12_D: now also U325.19 (OUT11); no longer U325.18 (OUT10)
- net DG12_E: now also U325.18 (OUT10); no longer U325.19 (OUT11)
- net DG13_B: now also U324.19 (OUT11); no longer U324.21 (OUT13)
- net DG13_C: now also U325.12 (OUT4); no longer U325.11 (OUT3)
- net DG13_D: now also U325.14 (OUT6); no longer U325.12 (OUT4)
- net DG13_DP: now also U325.11 (OUT3); no longer U325.10 (OUT2)
- net DG13_F: now also U324.18 (OUT10); no longer U324.19 (OUT11)
- net DG13_G: now also U324.17 (OUT9); no longer U324.18 (OUT10)
- net DG14_A: now also U329.10 (OUT2); no longer U329.9 (OUT1)
- net DG14_B: now also U329.9 (OUT1); no longer U329.10 (OUT2)
- net DG14_C: now also U330.22 (OUT14); no longer U330.23 (OUT15)
- net DG14_D: now also U325.10 (OUT2); no longer U325.8 (OUT0)
- net DG14_DP: now also U330.21 (OUT13); no longer U330.22 (OUT14)
- net DG14_F: now also U324.22 (OUT14); no longer U324.23 (OUT15)
- net DG14_G: now also U324.21 (OUT13); no longer U324.22 (OUT14)
- net DG15_A: now also U329.14 (OUT6); no longer U329.13 (OUT5)
- net DG15_B: now also U329.13 (OUT5); no longer U329.14 (OUT6)
- net DG15_D: now also U330.20 (OUT12); no longer U330.19 (OUT11)
- net DG15_E: now also U330.19 (OUT11); no longer U330.20 (OUT12)
- net DG16_A: now also U329.18 (OUT10); no longer U329.17 (OUT9)
- net DG16_B: now also U329.17 (OUT9); no longer U329.18 (OUT10)
- net DG16_D: now also U330.16 (OUT8); no longer U330.15 (OUT7)
- net DG16_E: now also U330.15 (OUT7); no longer U330.16 (OUT8)
- net DG17_A: now also U329.22 (OUT14); no longer U329.21 (OUT13)
- net DG17_B: now also U329.21 (OUT13); no longer U329.22 (OUT14)
- net DG17_D: now also U330.12 (OUT4); no longer U330.11 (OUT3)
- net DG17_E: now also U330.11 (OUT3); no longer U330.12 (OUT4)
- net DG18_A: now also U337.10 (OUT2); no longer U337.9 (OUT1)
- net DG18_B: now also U337.9 (OUT1); no longer U337.10 (OUT2)
- net DG18_D: now also U330.8 (OUT0); no longer U338.23 (OUT15)
- net DG18_E: now also U338.23 (OUT15); no longer U330.8 (OUT0)
- net DG19_A: now also U337.14 (OUT6); no longer U337.13 (OUT5)
- net DG19_B: now also U337.13 (OUT5); no longer U337.14 (OUT6)
- net DG19_D: now also U338.20 (OUT12); no longer U338.19 (OUT11)
- net DG19_E: now also U338.19 (OUT11); no longer U338.20 (OUT12)
- net DG1_A: now also U303.15 (OUT7); no longer U303.14 (OUT6)
- net DG1_B: now also U303.14 (OUT6); no longer U303.15 (OUT7)
- net DG1_D: now also U304.19 (OUT11); no longer U304.18 (OUT10)
- net DG1_E: now also U304.18 (OUT10); no longer U304.19 (OUT11)
- net DG20_A: now also U337.20 (OUT12); no longer U337.23 (OUT15)
- net DG20_C: now also U338.9 (OUT1); no longer U338.10 (OUT2)
- net DG20_DP: now also U338.8 (OUT0); no longer U338.9 (OUT1)
- net DG20_F: now also U337.16 (OUT8); no longer U337.15 (OUT7)
- net DG20_G: now also U337.17 (OUT9); no longer U337.16 (OUT8)
- net DG20_H: now also U337.18 (OUT10); no longer U337.17 (OUT9)
- net DG20_J: now also U337.21 (OUT13); no longer U337.20 (OUT12)
- net DG20_K: now also U337.23 (OUT15); no longer U337.21 (OUT13)
- net DG20_L: now also U338.10 (OUT2); no longer U338.11 (OUT3)
- net DG20_M: now also U338.11 (OUT3); no longer U338.12 (OUT4)
- net DG21_D: now also U338.12 (OUT4); no longer U338.8 (OUT0)
- net DG2_A: now also U303.19 (OUT11); no longer U303.18 (OUT10)
- net DG2_B: now also U303.18 (OUT10); no longer U303.19 (OUT11)
- net DG2_D: now also U304.15 (OUT7); no longer U304.14 (OUT6)
- net DG2_E: now also U304.14 (OUT6); no longer U304.15 (OUT7)
- net DG3_A: now also U303.23 (OUT15); no longer U303.22 (OUT14)
- net DG3_B: now also U303.22 (OUT14); no longer U303.23 (OUT15)
- net DG3_D: now also U304.11 (OUT3); no longer U304.10 (OUT2)
- net DG3_E: now also U304.10 (OUT2); no longer U304.11 (OUT3)
- net DG4_A: now also U311.11 (OUT3); no longer U311.10 (OUT2)
- net DG4_B: now also U311.10 (OUT2); no longer U311.11 (OUT3)
- net DG4_D: now also U312.23 (OUT15); no longer U312.22 (OUT14)
- net DG4_E: now also U312.22 (OUT14); no longer U312.23 (OUT15)
- net DG5_A: now also U311.15 (OUT7); no longer U311.14 (OUT6)
- net DG5_B: now also U311.14 (OUT6); no longer U311.15 (OUT7)
- net DG5_D: now also U312.19 (OUT11); no longer U312.18 (OUT10)
- net DG5_E: now also U312.18 (OUT10); no longer U312.19 (OUT11)
- net DG6_A: now also U311.19 (OUT11); no longer U311.18 (OUT10)
- net DG6_B: now also U311.18 (OUT10); no longer U311.19 (OUT11)
- net DG6_D: now also U312.15 (OUT7); no longer U312.14 (OUT6)
- net DG6_E: now also U312.14 (OUT6); no longer U312.15 (OUT7)
- net DG7_A: now also U311.23 (OUT15); no longer U311.22 (OUT14)
- net DG7_B: now also U311.22 (OUT14); no longer U311.23 (OUT15)
- net DG7_D: now also U312.11 (OUT3); no longer U312.10 (OUT2)
- net DG7_E: now also U312.10 (OUT2); no longer U312.11 (OUT3)
- net DG8_A: now also U317.11 (OUT3); no longer U317.10 (OUT2)
- net DG8_B: now also U317.10 (OUT2); no longer U317.11 (OUT3)
- net DG8_D: now also U318.23 (OUT15); no longer U318.22 (OUT14)
- net DG8_E: now also U318.22 (OUT14); no longer U318.23 (OUT15)
- net DG9_A: now also U317.15 (OUT7); no longer U317.14 (OUT6)
- net DG9_B: now also U317.14 (OUT6); no longer U317.15 (OUT7)
- net DG9_D: now also U318.19 (OUT11); no longer U318.18 (OUT10)
- net DG9_E: now also U318.18 (OUT10); no longer U318.19 (OUT11)
- net Earth: now also C329.1, C330.1, C331.1, C332.1, C333.1, C334.1

Commit message: update pcb
Parts:
- added C335, C336, C337: 1u, Capacitor_SMD:C_0402_1005Metric, symbol Device:C_Small
- added U346, U347, U348: 74AUP2G17, clock:XSON-6_SOT886, symbol Clock:74AUP2G17
Connections:
- net +3V3: now also C335.2, C336.2, C337.2, U346.5 (VDD), U347.5 (VDD), U348.5 (VDD)
- net Earth: now also C335.1, C336.1, C337.1, U346.2 (GND), U347.2 (GND), U348.2 (GND)
- net SEG_OE_MCU: now also U348.1 (1A); no longer U303.24 (OE), U304.24 (OE), U311.24 (OE), U312.24 (OE), U317.24 (OE), U318.24 (OE), U324.24 (OE), U325.24 (OE), U329.24 (OE), U330.24 (OE), U337.24 (OE), U338.24 (OE)
- new net SEG_OE_BF0: U329.24 (OE), U330.24 (OE), U337.24 (OE), U338.24 (OE), U347.1 (1A), U348.6 (1Y)
- new net SEG_OE_BF1: U317.24 (OE), U318.24 (OE), U324.24 (OE), U325.24 (OE), U346.1 (1A), U347.6 (1Y)
- new net SEG_OE_BF2: U303.24 (OE), U304.24 (OE), U311.24 (OE), U312.24 (OE), U346.6 (1Y)
- no-connect marks 5 -> 11
