File: kicad/GPS_CLock/GPS_CLock.kicad_sch (KiCad schematic)
At the start: 45 parts, among them J101 DEBUG, SW101 BOOT_JMP, SW102 BTN_UP, SW103 BTN_DWN, SW104 RUN, U101 W25Q16JVUXIQ, U102 VEML7700-TR, U103 RP2040

Commit message: update pcb
Parts:
- removed J101: DEBUG, Connector_PinHeader_2.54mm:PinHeader_1x10_P2.54mm_Vertical, symbol Connector_Generic:Conn_01x10
- removed R109, R111: 11k, Resistor_SMD:R_0402_1005Metric, symbol Device:R_Small
- removed R110, R112: 2.7k, Resistor_SMD:R_0402_1005Metric, symbol Device:R_Small
- added TP101, TP102, TP103, TP104, TP105, TP106, TP107, TP108, TP109, TP110: TestPoint, clock:MILLMAX_0531_PressFit, symbol Connector:TestPoint
Connections:
- net QC3.0 D-_GPIO1 is gone; now on net SEG_2.5V_TOP_EN: U103.2 (GPIO0)
- net +3V3: now also TP101.1
- net BATT_EN: now also U103.5 (GPIO3); no longer U103.7 (GPIO5)
- net BC_QON: now also U103.7 (GPIO5); no longer U103.5 (GPIO3)
- net Earth: now also TP102.1
- net GPS_PPS: now also TP110.1
- net GPS_RX: now also TP109.1
- net GPS_TX: now also TP108.1
- net RUN: now also TP103.1
- net SEG_2.5V_TOP_EN: no longer U103.41 (GPIO29_ADC3)
- net SWCLK: now also TP105.1
- net SWD: now also TP104.1
- net UART_RX: now also TP107.1
- net UART_TX: now also TP106.1
- net DM-D+ renamed MCU-D-
- net DM-D- renamed MCU-D+
- net QC3.0 D+_GPIO: no longer names the net of U103.4 (GPIO2)
- net QC3.0 D-_GPIO0: no longer names the net of U103.3 (GPIO1)
- net USB-D+: no longer names the net of R104.2, U103.46 (USB_DM)
- net USB-D-: no longer names the net of R103.2, U103.47 (USB_DP)
- no-connect marks 0 -> 3
Other:
- sheet Power ports: added MCU-D+, MCU-D-; removed DM-D+, DM-D-
- moved on the sheet: R103, R104

Commit message: update pcb
Parts:
- added R109: 100k, Resistor_SMD:R_0402_1005Metric, symbol Device:R_Small
Connections:
- net SEG_2.5V_BOT_EN is gone; now on net DISP_RST: U103.14 (GPIO11)
- net BATT_EN: now also U103.4 (GPIO2); no longer U103.5 (GPIO3)
- net BC_INT: now also U103.5 (GPIO3); no longer U103.6 (GPIO4)
- net BC_QON: now also U103.6 (GPIO4); no longer U103.7 (GPIO5)
- net BTN_DWN: now also U103.18 (GPIO15); no longer U103.29 (GPIO18)
- net BTN_UP: now also U103.16 (GPIO13); no longer U103.30 (GPIO19)
- net DISP_BL: now also U103.17 (GPIO14); no longer U103.18 (GPIO15)
- net DISP_CLK: now also U103.12 (GPIO9); no longer U103.13 (GPIO10)
- net DISP_COPI: now also U103.11 (GPIO8); no longer U103.12 (GPIO9)
- net DISP_CS: now also U103.15 (GPIO12); no longer U103.17 (GPIO14)
- net DISP_DC: now also U103.13 (GPIO10); no longer U103.15 (GPIO12)
- net DISP_RST: no longer U103.16 (GPIO13)
- net Earth: now also R109.2
- net PD_INT: now also U103.9 (GPIO7); no longer U103.11 (GPIO8)
- net POW_SCL: now also U103.8 (GPIO6); no longer U103.9 (GPIO7)
- net POW_SDA: now also U103.7 (GPIO5); no longer U103.8 (GPIO6)
- net SEG_CLK: now also U103.31 (GPIO20); no longer U103.34 (GPIO22)
- net SEG_LAT: now also U103.30 (GPIO19); no longer U103.32 (GPIO21)
- net SEG_MOSI: now also U103.29 (GPIO18); no longer U103.31 (GPIO20)
- net SEG_OE: now also U103.32 (GPIO21); no longer U103.35 (GPIO23)
- net SEG_2.5V_TOP_EN renamed 2V5_EN
- net 2V5_EN: now also R109.1
- no-connect marks 3 -> 2

Commit message: modify pcb
Connections:
- net USB_SW: now reaches U103.3 (GPIO1)
- no-connect marks 2 -> 3
Other:
- sheet Power ports: added FG_SCL, FG_SDA, USB_SW; removed none
Changed lines of the file:
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@@
   (junction (at 80.01 165.1) (diameter 0) (color 0 0 0 0)
   )
-  (junction (at 163.83 43.18) (diameter 0) (color 0 0 0 0)
-  )
   (junction (at 170.18 35.56) (diameter 0) (color 0 0 0 0)
   )
@@
   )
   (no_connect (at 163.83 119.38))
-  (no_connect (at 163.83 45.72))
+  (no_connect (at 163.83 99.06))
+  (no_connect (at 163.83 101.6))
   (wire (pts (xy 53.34 124.46) (xy 49.53 124.46))
     (stroke (width 0) (type default) (color 0 0 0 0))
@@
     (stroke (width 0) (type default) (color 0 0 0 0))
   )
+  (wire (pts (xy 177.8 45.72) (xy 163.83 45.72))
+    (stroke (width 0) (type default) (color 0 0 0 0))
+  )
   (wire (pts (xy 27.94 67.31) (xy 22.86 67.31))
     (stroke (width 0) (type default) (color 0 0 0 0))
@@
     (stroke (width 0) (type default) (color 0 0 0 0))
   )
-  (wire (pts (xy 160.02 43.18) (xy 163.83 43.18))
-    (stroke (width 0) (type default) (color 0 0 0 0))
-  )
   (wire (pts (xy 163.83 76.2) (xy 177.8 76.2))
     (stroke (width 0) (type default) (color 0 0 0 0))
@@
     (stroke (width 0) (type default) (color 0 0 0 0))
   )
+  (wire (pts (xy 229.87 127) (xy 243.84 127))
+    (stroke (width 0) (type default) (color 0 0 0 0))
+  )
   (wire (pts (xy 43.18 124.46) (xy 49.53 124.46))
     (stroke (width 0) (type default) (color 0 0 0 0))
@@
     (stroke (width 0) (type default) (color 0 0 0 0))
   )
+  (wire (pts (xy 229.87 121.92) (xy 243.84 121.92))
+    (stroke (width 0) (type default) (color 0 0 0 0))
+  )
   (wire (pts (xy 80.01 165.1) (xy 80.01 166.37))
     (stroke (width 0) (type default) (color 0 0 0 0))
@@
     (stroke (width 0) (type default) (color 0 0 0 0))
   )
+  (wire (pts (xy 229.87 129.54) (xy 243.84 129.54))
+    (stroke (width 0) (type default) (color 0 0 0 0))
+  )
   (wire (pts (xy 228.6 163.83) (xy 237.49 163.83))
     (stroke (width 0) (type default) (color 0 0 0 0))
@@
     (effects (font (size 1.27 1.27)) (justify left bottom))
   )
+  (label "USB_SW" (at 177.8 45.72 180)
+    (effects (font (size 1.27 1.27)) (justify right bottom))
+  )
   (label "QSPI_SD0" (at 101.6 66.04 0)
     (effects (font (size 1.27 1.27)) (justify left bottom))
@@
     (effects (font (size 1.27 1.27)) (justify left bottom))
   )
+  (label "USB_SW" (at 229.87 121.92 0)
+    (effects (font (size 1.27 1.27)) (justify left bottom))
+  )
   (label "UART_TX" (at 177.8 86.36 180)
     (effects (font (size 1.27 1.27)) (justify right bottom))
@@
     (effects (font (size 1.27 1.27)) (justify right bottom))
   )
+  (label "SEN_SCL" (at 229.87 127 0)
+    (effects (font (size 1.27 1.27)) (justify left bottom))
+  )
   (label "BATT_EN" (at 229.87 93.98 0)
     (effects (font (size 1.27 1.27)) (justify left bottom))
@@
     (effects (font (size 1.27 1.27)) (justify left bottom))
   )
+  (label "SEN_SDA" (at 229.87 129.54 0)
+    (effects (font (size 1.27 1.27)) (justify left bottom))
+  )
   (label "SEN_SCL" (at 177.8 114.3 180)
     (effects (font (size 1.27 1.27)) (justify right bottom))
@@
     (pin "9")
   )
-  (sheet (at 243.84 80.01) (size 19.05 41.91) (fields_autoplaced)
+  (sheet (at 243.84 80.01) (size 19.05 53.34) (fields_autoplaced)
     (stroke (width 0.1524) (type solid) (color 0 0 0 0))
     (fill (color 0 0 0 0.0000))
@@
       (effects (font (size 1.27 1.27)) (justify left bottom))
     )
-    (property "Sheet file" "Power.kicad_sch" (id 1) (at 243.84 122.5046 0)
+    (property "Sheet file" "Power.kicad_sch" (id 1) (at 243.84 133.9346 0)
       (effects (font (size 1.27 1.27)) (justify left top) hide)
     )
@@
       (effects (font (size 1.27 1.27)) (justify left))
     )
+    (pin "FG_SCL" input (at 243.84 127 180)
+      (effects (font (size 1.27 1.27)) (justify left))
+    )
+    (pin "FG_SDA" input (at 243.84 129.54 180)
+      (effects (font (size 1.27 1.27)) (justify left))
+    )
+    (pin "USB_SW" input (at 243.84 121.92 180)
+      (effects (font (size 1.27 1.27)) (justify left))
+    )
   )
   (sheet (at 207.01 104.14) (size 12.7 17.78) (fields_autoplaced)
@@
       (reference "#PWR0134") (unit 1) (value "+3V3") (footprint "")
     )
+    (path "/1f693c02-7734-4d07-85c5-22483e243ef7/173cd01a-e5d4-4742-9356-d3d61817c6b3"
+      (reference "#PWR0135") (unit 1) (value "Earth") (footprint "")
+    )
+    (path "/1f693c02-7734-4d07-85c5-22483e243ef7/b154a664-efb0-4e06-a3f6-2fec65b92112"
+      (reference "#PWR0136") (unit 1) (value "Earth") (footprint "")
+    )
+    (path "/1f693c02-7734-4d07-85c5-22483e243ef7/200d4b6c-2e4a-40dd-8ff2-4b83d2ea0278"
+      (reference "#PWR0137") (unit 1) (value "Earth") (footprint "")
+    )
+    (path "/1f693c02-7734-4d07-85c5-22483e243ef7/4855b5b1-3f5a-46d2-b917-7bca685a51c7"
+      (reference "#PWR0138") (unit 1) (value "Earth") (footprint "")
+    )
+    (path "/1f693c02-7734-4d07-85c5-22483e243ef7/496399a7-0b72-4433-a057-e245002435c8"
+      (reference "#PWR0139") (unit 1) (value "Earth") (footprint "")
+    )
+    (path "/1f693c02-7734-4d07-85c5-22483e243ef7/ab0cb75f-c4db-4911-a49f-a4538f98bdc4"
+      (reference "#PWR0140") (unit 1) (value "Earth") (footprint "")
+    )
     (path "/4fbde836-87d5-478f-8d01-f08e4241a9c4/11abb5d0-9c5a-43e7-9733-c1460163c319"
       (reference "#PWR0162") (unit 1) (value "Earth") (footprint "")
@@
       (reference "#PWR0316") (unit 1) (value "Earth") (footprint "")
     )
-    (path "/1f693c02-7734-4d07-85c5-22483e243ef7/7edd453b-f6f9-404d-b6a2-aa56146267a3"
-      (reference "#PWR0317") (unit 1) (value "+BATT") (footprint "")
-    )
-    (path "/1f693c02-7734-4d07-85c5-22483e243ef7/dfb55799-1391-471d-b190-9dcecb42bda1"
-      (reference "#PWR0318") (unit 1) (value "Earth") (footprint "")
-    )
     (path "/1f693c02-7734-4d07-85c5-22483e243ef7/092d92a5-2694-459b-bed6-1b9c6b506a14"
       (reference "#PWR0319") (unit 1) (value "Earth") (footprint "")
     )
-    (path "/1f693c02-7734-4d07-85c5-22483e243ef7/ff8e6c56-4728-4704-88b9-657a3014f63f"
-      (reference "#PWR0320") (unit 1) (value "Earth") (footprint "")
-    )
-    (path "/1f693c02-7734-4d07-85c5-22483e243ef7/ff4e7dc1-2241-4656-8db8-0a1b74a7a27e"
-      (reference "#PWR0321") (unit 1) (value "Earth") (footprint "")
-    )
     (path "/1f693c02-7734-4d07-85c5-22483e243ef7/46f45ce8-ffcb-4f0d-b6d5-ac1be2a8b9b7"
       (reference "#PWR0322") (unit 1) (value "Earth") (footprint "")
@@
       (reference "C236") (unit 1) (value "1n") (footprint "Capacitor_SMD:C_0402_1005Metric")
     )
+    (path "/1f693c02-7734-4d07-85c5-22483e243ef7/0ca30340-627e-4ff1-b809-dc5de0f2ee2c"
+      (reference "C237") (unit 1) (value "0.1u") (footprint "Capacitor_SMD:C_0402_1005Metric")
+    )
     (path "/4fbde836-87d5-478f-8d01-f08e4241a9c4/f1fceaca-23b9-4e18-a949-86ee054a348a"
       (reference "C301") (unit 1) (value "1u") (footprint "Capacitor_SMD:C_0402_1005Metric")
@@
       (reference "R115") (unit 1) (value "10k") (footprint "Resistor_SMD:R_0402_1005Metric")
     )
+    (path "/1f693c02-7734-4d07-85c5-22483e243ef7/5111df16-7ea7-4379-9a8f-b3f4c83a0af2"
+      (reference "R201") (unit 1) (value "10m") (footprint "Resistor_SMD:R_2512_6332Metric")
+    )
     (path "/1f693c02-7734-4d07-85c5-22483e243ef7/67206d1d-0475-4b4b-899d-3482d5ab17bb"
       (reference "R203") (unit 1) (value "100k") (footprint "Resistor_SMD:R_0402_1005Metric")
@@
       (reference "U206") (unit 1) (value "USB3740B-AI2") (footprint "Package_DFN_QFN:UQFN-10_1.3x1.8mm_P0.4mm")
     )
+    (path "/1f693c02-7734-4d07-85c5-22483e243ef7/1b289f6d-a96b-42f3-8b94-cd61043735fe"
+      (reference "U207") (unit 1) (value "LTC2942") (footprint "Package_DFN_QFN:DFN-6-1EP_3x2mm_P0.5mm_EP1.65x1.35mm")
+    )
     (path "/4fbde836-87d5-478f-8d01-f08e4241a9c4/b9c95ca2-a7b1-44de-9f8d-f4ea8d9de37b"
