File: kicad/GPS_CLock/Power.kicad_sch (KiCad schematic)
At the start: 72 parts, among them J201 USB_C_2.0, U201 TPS62827DMQ, U202 TPS62827DMQ, U203 FUSB302BMPX, U204 BQ25792RQM, U205 LP5912-3.3DRV

Commit message: update pcb
Parts:
- added C236: 1n, Capacitor_SMD:C_0402_1005Metric, symbol Device:C_Small
- added R220: 100k, Resistor_SMD:R_0402_1005Metric, symbol Device:R_Small
- added U206: USB3740B-AI2, Package_DFN_QFN:UQFN-10_1.3x1.8mm_P0.4mm, symbol Interface_USB:USB3740B-AI2
Connections:
- net +3V3: now also C236.2, U206.5 (VDD)
- net Earth: now also C236.1, R220.2, U206.3 (OE_N), U206.8 (GND)
- net BC-D+: now reaches U204.6 (D+)
- net BC-D+: now also U206.6 (DP_2)
- net BC-D-: now reaches U204.7 (D-)
- net BC-D-: now also U206.7 (DM_2)
- net DM-D+ renamed CON-D+
- net CON-D+: now also U206.9 (DM)
- net DM-D- renamed CON-D-
- net CON-D-: now also U206.10 (DP)
- new net MCU-D+: U206.1 (DM_1)
- new net MCU-D-: U206.2 (DP_1)
- new net USB_SW: R220.1, U206.4 (S)
- no-connect marks 4 -> 2
Other:
- moved on the sheet: C203, C204, C205, C208, C209, C214, C216, C218, C220, C221, U203
