File: kicad/GPS_CLock/Power.kicad_sch (KiCad schematic)
At the start: 75 parts, among them J201 USB_C_2.0, U201 TPS62827DMQ, U202 TPS62827DMQ, U203 FUSB302BMPX, U204 BQ25792RQM, U205 LP5912-3.3DRV, U206 USB3740B-AI2

Commit message: update pcb
Parts:
- removed R201, R202: 100k, Resistor_SMD:R_0402_1005Metric, symbol Device:R_Small
Other:
- moved on the sheet: C201, C202

Commit message: modify pcb
Parts:
- added C237: 0.1u, Capacitor_SMD:C_0402_1005Metric, symbol Device:C_Small
- added R201: 10m, Resistor_SMD:R_2512_6332Metric, symbol Device:R_Small
- added U207: LTC2942, Package_DFN_QFN:DFN-6-1EP_3x2mm_P0.5mm_EP1.65x1.35mm, symbol Battery_Management:LTC2942
Connections:
- net Earth: now also C237.2, U207.2 (GND), U207.5 (~{AL}/CC)
- net +BATT renamed SENSE+
- net SENSE+: now also C237.1, R201.1, U207.1 (SENSE+); no longer BT201.1 (+), JP201.2 (B), R217.1
- new net FG_SCL: U207.3 (SCL)
- new net FG_SDA: U207.4 (SDA)
- new net SENSE-: BT201.1 (+), JP201.2 (B), R201.2, R217.1, U207.6 (SENSE-)
Other:
- moved on the sheet: BT201, BT202, BT203, C227, C228, C230, C231, C232, C233, C234, C235, JP201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
